Commit message: Done writing urdf parser

File: lbr_iiwa/urdf/lbr_iiwa_meshfree.urdf (robot description, URDF)
Before this commit: robot lbr_iiwa, 5 links, 4 joints
Links:
- added link lbr_iiwa_end_effector
Joints:
- added joint lbr_iiwa_joint_4: type fixed, parent lbr_iiwa_link_3, child lbr_iiwa_end_effector, origin xyz=0 0 0.2155 rpy=0 0 0, axis 0 0 1, limit lower=-2.96705972839 upper=2.96705972839 effort=10 velocity=10
- joint lbr_iiwa_joint_1: origin xyz=0 0 0.1575 rpy=0 0 1 -> xyz=0 0 0.1575 rpy=0 0 0
- joint world_joint: origin xyz=0 0 0 rpy=0 0 0 -> xyz=0 0 0.0 rpy=0 0 0

File: lbr_iiwa/urdf/lbr_iiwa_meshfree_simple.xacro (robot description, xacro)
@@ -164,4 +164,20 @@
       </collision>
     </link>
+    <joint name="${name}_joint_4" type="fixed">
+      <parent link="${name}_link_3"/>
+      <child link="${name}_end_effector"/>
+      <origin xyz="0 0 ${len_link_3}" rpy="0 0 0"/>
+      <axis xyz="0 0 1"/>
+      <limit lower="${-170 * PI / 180}" upper="${170 * PI / 180}"
+             effort="${max_effort_joint3}" velocity="${max_velocity}" />
+      <!--limit lower="0" upper="0"
+             effort="${max_effort_joint3}" velocity="${max_velocity}" /-->
+      <!-- <safety_controller soft_lower_limit="${-118 * PI / 180}"
+           soft_upper_limit="${118 * PI / 180}"
+           k_position="${safety_controller_k_pos}"
+           k_velocity="${safety_controller_k_vel}"/> -->
+      <dynamics damping="${joint_damping}"/>
+    </joint>
+    <link name="${name}_end_effector"/>
     <!--Extensions -->
     <xacro:lbr_iiwa_gazebo name="${name}" />
