Commit message: am

File: test.urdf (robot description, URDF)
Before this commit: robot lbr_iiwa, 4 links, 3 joints
Links:
- added link link3, mass 5; collision box size=1 0.15 0.15; visual box size=1 0.15 0.15
Joints:
- added joint joint4: type revolute, parent link3, child end_effector, origin xyz=1 0 0 rpy=0 0 0, axis 0 0 1, limit lower=-3.14159265359 upper=3.14159265359 effort=10 velocity=10
- joint joint3: child end_effector -> link3

Commit message: Changes

File: test.urdf (robot description, URDF)
Before this commit: robot lbr_iiwa, 5 links, 4 joints
Links:
- removed link link3
Joints:
- removed joint joint4
- joint joint3: child link3 -> end_effector

Commit message: Fixes to code generation

File: test.urdf (robot description, URDF)
Before this commit: robot lbr_iiwa, 4 links, 3 joints
Joints:
- joint joint1: origin xyz=1 0 0 rpy=0 0 0 -> xyz=1 0 1 rpy=0 0 0

Commit message: Bugfixing

File: test.urdf (robot description, URDF)
Before this commit: robot lbr_iiwa, 4 links, 3 joints
Links:
- link link2: mass 5 -> 50
Joints:
- joint joint1: origin xyz=1 0 1 rpy=0 0 0 -> xyz=0 0 5 rpy=-1.57079632679489661923 0 0

Commit message: Bugfixing

File: test.urdf (robot description, URDF)
Before this commit: robot lbr_iiwa, 4 links, 3 joints
Links:
- link link2: mass 50 -> 5
